File: switched_usb_hub.kicad_pcb (KiCad board)
At the start: 2 copper layers, 51 x 71 mm, 56 parts, among them J1 USB_C_Receptacle_USB2.0, J2 USB_A, J3 USB_A, J4 USB_A, J5 JTAG_CONN, Q1 IRLML6402, Q2 IRLML6402, Q3 IRLML6402, U1 SL2.1A, U2 CH340C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

Commit message: adding rev A hopefully final files
Other:
- rule pad_to_mask_clearance: 0 -> 0.05
- board text added: "OUT1"
- board text added: "OUT2"
- board text added: "OUT3"
